Commit message: IMU added to URDF

File: sahayak/urdf/sahayak.urdf (robot description, URDF)
Before this commit: robot sahayak, 12 links, 11 joints
Links:
- added link imu_link
Joints:
- added joint imu_joint: type fixed, parent base_link, child imu_link

Commit message: Updated URDF and added mapping launch files

File: sahayak/urdf/sahayak.urdf (robot description, URDF)
Before this commit: robot sahayak, 13 links, 12 joints
Links:
- added link pseudo_base
- link imu_link: mass None -> 0.001; geometry visual box size=0.001 0.001 0.001
- link rplidar: mass None -> 0.19; geometry visual box size=0.02 0.05 0.05
Joints:
- added joint base2base_joint: type fixed, parent base_link, child pseudo_base, origin xyz=0 0 0 rpy=1.54 1.54 0
- joint imu_joint: origin (none) -> xyz=0 0 0 rpy=1.57 0 0

Commit message: Added ROS Navigation to Sahayak

File: sahayak/urdf/sahayak.urdf (robot description, URDF)
Before this commit: robot sahayak, 14 links, 13 joints
Links:
- removed link pseudo_base
Joints:
- removed joint Lidar1
- removed joint base2base_joint
- added joint Lidar_J: type fixed, parent base_link, child Lidar, origin xyz=0 -0.4025 0.9125 rpy=1.5708 0 1.5469, axis 0 1 0, limit lower=0 upper=0 effort=0 velocity=0
- joint Wheel_left_back_J: limit lower=0 upper=0 effort=0.67 velocity=6.28 -> lower=0 upper=0 effort=1 velocity=6.28; origin xyz=-0.21192 0.025 -0.1875 rpy=1.5708 0 0 -> xyz=-0.21192 -0.35 0.085 rpy=1.5708 0 0
- joint Wheel_left_front_J: limit lower=0 upper=0 effort=0.67 velocity=6.28 -> lower=0 upper=0 effort=1 velocity=6.28; origin xyz=-0.21342 0.025 0.1875 rpy=1.5708 0 0 -> xyz=-0.21342 0.025 0.085 rpy=1.5708 0 0
- joint Wheel_right_back_J: axis -1 0 0 -> 1 0 0; limit lower=0 upper=0 effort=0.67 velocity=6.28 -> lower=0 upper=0 effort=1 velocity=6.28; origin xyz=0.21192 0.025 -0.1875 rpy=1.5708 0 0 -> xyz=0.21192 -0.35 0.085 rpy=1.5708 0 3.1416
- joint Wheel_right_front_J: axis -1 0 0 -> 1 0 0; limit lower=0 upper=0 effort=0.67 velocity=6.28 -> lower=0 upper=0 effort=1 velocity=6.28; origin xyz=0.21342 0.025 0.1875 rpy=1.5708 0 0 -> xyz=0.21342 0.025 0.085 rpy=1.5708 0 3.1416
- joint realsense_joint: origin xyz=1.1752E-05 -0.54426 0.237 rpy=0 -1.570 1.570 -> xyz=1.1752E-05 0.0745 0.65426 rpy=0 0 1.57
- joint rplidar_joint: origin xyz=0 -0.8025 -0.24 rpy=1.570 1.5469 0 -> xyz=0 -0.4025 0.9125 rpy=3.14 0 1.5469
